Commit message: add bluerov2 with hdt arm

File: bluerov2_description/urdf/base.xacro (robot description, xacro)
@@ -72,10 +72,10 @@
         </visual>
         <!-- In rexrov2_base they made collision planes to minize the GPU load -->
-        <!-- <collision>
+        <collision>
           <origin xyz="0 0 0" rpy="0 0 0"/>
           <geometry>
             <mesh filename="${collision_mesh_file}" scale="1 1 1" />
           </geometry>
-        </collision> -->
+        </collision>
       </link>
     <gazebo reference="${namespace}/base_link">
